File: Hardware/PCB_Design/ComputationalPrototype.kicad_pcb (KiCad board)
At the start: 2 copper layers, 56 parts, among them IC1 PCF8523T_1,118, IC2 1072, J1 Conn_02x20_Odd_Even, J2 Screw_Terminal_01x02, J3 Screw_Terminal_01x05, J4 USB_B_Micro, J5 ISP Header, Q1 FQP_27P06, Q2 2N3904, SW1 SW_Push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

Commit message: Add files via upload
Parts:
- C4: value 1uF -> 100uF
- moved J2 2.54 mm to (142.5, 64.6), turned to 180 degrees
Connections:
- U2 pad 1: Net-(IC1-Pad7) -> Net-(U2-Pad1)
- Y2 pad 1: Net-(IC1-Pad1) -> Net-(Y2-Pad1)
- Y2 pad 2: Net-(IC1-Pad2) -> Net-(Y2-Pad2)
Routing:
- net +12V: track 16.5 -> 17.6 mm

Commit message: Add files via upload
Parts:
- added JP1: SNT-100-YW-T, Connector_PinHeader_2.54mm:PinHeader_1x02_P2.54mm_Vertical, F.Cu at (158.0, 100.2)
- D1, D2, D3: value LED_ALT -> 151031VS06000
- J1: value Conn_02x20_Odd_Even -> PinSocket_2x20_P2.54mm_Vertical
- J2: value Screw_Terminal_01x02 -> 1725656
- J3: value Screw_Terminal_01x05 -> 1725685
- J5: value ISP Header -> PinHeader_2x03_P2.54mm_Vertical
- Q1: value FQP_27P06 -> FQP27P06
- SW1, SW2: value SW_Push -> PTS645SL432LFS
- SW3: value SW_DIP_x02 -> 1825057-1
- U1: value MCP1703A-3302_SOT23 -> MCP1703AT-3302E/CB
- U4: value 25LCxxx -> 25LC1024-E/SM
- U5: value 74125 -> SN74HC125DR
- Y1: value 8MHz -> F90800021
- Y2: value 32.768kHz -> LFXTAL050789REEL
- moved J3 10.2 mm to (135.6, 64.6), turned to 180 degrees
Connections:
- IC1 pad 6: Net-(J3-Pad2) -> Net-(J3-Pad4)
- J3 pad 1: Net-(J3-Pad1) -> +3V3
- J3 pad 2: Net-(J3-Pad2) -> GND
- J3 pad 4: GND -> Net-(J3-Pad4)
- J3 pad 5: +3V3 -> Net-(J3-Pad5)
- R3 pad 2: Net-(J3-Pad2) -> Net-(J3-Pad4)
- U2 pad 28: Net-(J3-Pad2) -> Net-(J3-Pad4)
- U2 pad 32: Net-(J3-Pad1) -> Net-(J3-Pad5)
- U4 pad 3: +3V3 -> VCC
- U4 pad 7: +3V3 -> VCC
- U4 pad 8: +3V3 -> VCC
Routing:
- net Net-(J3-Pad4): track 0.00 -> 54.4 mm
- net Net-(J3-Pad2): track 54.4 -> 0.00 mm
- net Net-(J3-Pad5): track 0.00 -> 53.3 mm, vias 0 -> 1
- net Net-(J3-Pad1): track 53.3 -> 0.00 mm, vias 1 -> 0
- net VCC: track 2.08 -> 30.3 mm, vias 1 -> 3
- net Net-(J5-Pad4): track 45.9 -> 35.2 mm
- net +3V3: track 46.3 -> 41.7 mm, vias 4 -> 2
- net Net-(J5-Pad1): track 48.3 -> 45.1 mm
Other:
- board outline added: 56.5 x 64.8 mm
- board text added: "EEPROM Power"
