File: Hardware/PCB_Design/ComputationalPrototype.kicad_pcb (KiCad board)
At the start: 2 copper layers, 56 parts, among them IC1 PCF8523T_1,118, IC2 1072, J1 Conn_02x20_Odd_Even, J2 Screw_Terminal_01x02, J3 Screw_Terminal_01x05, J4 USB_B_Micro, J5 ISP Header, Q1 FQP_27P06, Q2 2N3904, SW1 SW_Push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

Commit message: Add files via upload
Parts:
- D1, D2, D3: value LED_ALT -> 2460-L314HD-ND
- SW1, SW2: value SW_Push -> 611-PTS645SL43SMTR92
- SW3: value SW_DIP_x02 -> 1825057-1
- U4: value 25LCxxx -> 25LC1024-E/SM
- U5: value 74125 -> SN74HC125D
- Y1: value 8MHz -> F90800021
- Y2: value 32.768kHz -> LFXTAL050789REEL
- moved Q2 11.8 mm to (146.1, 84.8), turned to 0 degrees
- moved C3 10.1 mm to (146.7, 64.6), turned to 0 degrees
- moved R10 8.84 mm to (141.1, 83.3)
- moved R11 8.84 mm to (138.5, 83.3)
- moved Q1 8.49 mm to (148.8, 77.0)
- moved R2 6.55 mm to (146.7, 66.9)
Routing:
- net Net-(Q1-Pad1): track 10.3 -> 20.0 mm
- net GND: track 65.3 -> 74.5 mm, vias 3 -> 5
- net Net-(J1-Pad18): track 52.8 -> 46.9 mm
- net Net-(R10-Pad2): track 28.6 -> 22.9 mm
- net Net-(J1-Pad22): track 61.4 -> 56.5 mm
- net +12V: track 16.5 -> 19.3 mm
- net Net-(Q2-Pad2): track 5.79 -> 7.98 mm
- net +3V3: track 46.3 -> 48.4 mm, vias 4 -> 5
- net Net-(C15-Pad1): track 16.1 -> 15.6 mm
Other:
- board outline added: 56.6 x 64.9 mm
- board text added: "12V"
- board text added: "3V3"
- board text added: "BRN"
- board text added: "GND"
- board text added: "GRN"
- board text added: "WHT"

Commit message: Add files via upload
Parts:
- D1, D2, D3: value 2460-L314HD-ND -> LED_ALT
- SW1, SW2: value 611-PTS645SL43SMTR92 -> SW_Push
- SW3: value 1825057-1 -> SW_DIP_x02
- U4: value 25LC1024-E/SM -> 25LCxxx
- U5: value SN74HC125D -> 74125
- Y1: value F90800021 -> 8MHz
- Y2: value LFXTAL050789REEL -> 32.768kHz
- moved Q2 11.8 mm to (150.9, 74.0), turned to 180 degrees
- moved C3 10.1 mm to (141.4, 73.3), turned to 90 degrees
- moved R10 8.84 mm to (149.6, 80.8)
- moved R11 8.84 mm to (147.0, 80.8)
- moved Q1 8.49 mm to (148.3, 68.5)
- moved R2 6.55 mm to (144.7, 73.2)
Routing:
- net Net-(Q1-Pad1): track 20.0 -> 10.3 mm
- net GND: track 74.5 -> 65.3 mm, vias 5 -> 3
- net Net-(J1-Pad18): track 46.9 -> 52.8 mm
- net Net-(R10-Pad2): track 22.9 -> 28.6 mm
- net Net-(J1-Pad22): track 56.5 -> 61.4 mm
- net +12V: track 19.3 -> 16.5 mm
- net Net-(Q2-Pad2): track 7.98 -> 5.79 mm
- net +3V3: track 48.4 -> 46.3 mm, vias 5 -> 4
- net Net-(C15-Pad1): track 15.6 -> 16.1 mm
Other:
- board outline removed
- board text removed: "12V"
- board text removed: "3V3"
- board text removed: "BRN"
- board text removed: "GND"
- board text removed: "GRN"
- board text removed: "WHT"

Commit message: Add files via upload
Parts:
- added JP1: Jumper_2_Bridged, Connector_PinHeader_2.54mm:PinHeader_1x02_P2.54mm_Vertical, F.Cu at (158.0, 100.2)
- C4: value 1uF -> 100uF
- SW1, SW2: value SW_Push -> PTS645SL432LFS
- U1: value MCP1703A-3302_SOT23 -> MCP1703AT-3302E/CB
- moved J3 10.2 mm to (135.6, 64.6), turned to 180 degrees
- moved J2 2.54 mm to (142.5, 64.6), turned to 180 degrees
Connections:
- IC1 pad 6: Net-(IC1-Pad6) -> Net-(J3-Pad4)
- J3 pad 1: Net-(J3-Pad1) -> +3V3
- J3 pad 2: Net-(IC1-Pad6) -> GND
- J3 pad 4: GND -> Net-(J3-Pad4)
- J3 pad 5: +3V3 -> Net-(J3-Pad5)
- R3 pad 2: Net-(IC1-Pad6) -> Net-(J3-Pad4)
- U2 pad 1: Net-(IC1-Pad7) -> Net-(U2-Pad1)
- U2 pad 28: Net-(IC1-Pad6) -> Net-(J3-Pad4)
- U2 pad 32: Net-(J3-Pad1) -> Net-(J3-Pad5)
- U4 pad 3: +3V3 -> VCC
- U4 pad 7: +3V3 -> VCC
- U4 pad 8: +3V3 -> VCC
- Y2 pad 1: Net-(IC1-Pad1) -> Net-(Y2-Pad1)
- Y2 pad 2: Net-(IC1-Pad2) -> Net-(Y2-Pad2)
Routing:
- net Net-(J3-Pad4): track 0.00 -> 54.4 mm
- net Net-(IC1-Pad6): track 54.4 -> 0.00 mm
- net Net-(J3-Pad5): track 0.00 -> 53.3 mm, vias 0 -> 1
- net Net-(J3-Pad1): track 53.3 -> 0.00 mm, vias 1 -> 0
- net VCC: track 2.08 -> 30.3 mm, vias 1 -> 3
- net Net-(J5-Pad4): track 45.9 -> 35.2 mm
- net +3V3: track 46.3 -> 41.7 mm, vias 4 -> 2
- net Net-(J5-Pad1): track 48.3 -> 45.1 mm
- net +12V: track 16.5 -> 17.6 mm
Other:
- board outline added: 56.5 x 64.8 mm
- board text added: "EEPROM Power"

Commit message: Add files via upload
Parts:
- D1, D2, D3: value LED_ALT -> 151031VS06000
- J1: value Conn_02x20_Odd_Even -> PinSocket_2x20_P2.54mm_Vertical
- J2: value Screw_Terminal_01x02 -> 1725656
- J3: value Screw_Terminal_01x05 -> 1725685
- J5: value ISP Header -> PinHeader_2x03_P2.54mm_Vertical
- JP1: value Jumper_2_Bridged -> SNT-100-YW-T
- Q1: value FQP_27P06 -> FQP27P06
- SW3: value SW_DIP_x02 -> 1825057-1
- U4: value 25LCxxx -> 25LC1024-E/SM
- U5: value 74125 -> SN74HC125DR
- Y1: value 8MHz -> F90800021
- Y2: value 32.768kHz -> LFXTAL050789REEL
Changed lines of the file:
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@@
       (effects (font (size 1 1) (thickness 0.15)))
     )
-    (fp_text value Jumper_2_Bridged (at 0 4.87 90) (layer F.Fab)
+    (fp_text value SNT-100-YW-T (at 0 4.87 90) (layer F.Fab)
       (effects (font (size 1 1) (thickness 0.15)))
     )
@@
       (effects (font (size 1 1) (thickness 0.15)))
     )
-    (fp_text value 74125 (at 0 5.375) (layer F.Fab)
+    (fp_text value SN74HC125DR (at 0 5.375) (layer F.Fab)
       (effects (font (size 1 1) (thickness 0.15)))
     )
@@
       (effects (font (size 1 1) (thickness 0.15)))
     )
-    (fp_text value LED_ALT (at 1.27 2.96) (layer F.Fab)
+    (fp_text value 151031VS06000 (at 1.27 2.96) (layer F.Fab)
       (effects (font (size 1 1) (thickness 0.15)))
     )
@@
       (effects (font (size 1 1) (thickness 0.15)))
     )
-    (fp_text value LED_ALT (at 1.25 0 90) (layer F.Fab)
+    (fp_text value 151031VS06000 (at 1.25 0 90) (layer F.Fab)
       (effects (font (size 1 1) (thickness 0.15)))
     )
@@
       (effects (font (size 1 1) (thickness 0.15)))
     )
-    (fp_text value LED_ALT (at 1.27 0 90) (layer F.Fab)
+    (fp_text value 151031VS06000 (at 1.27 0 90) (layer F.Fab)
       (effects (font (size 1 1) (thickness 0.15)))
     )
@@
       (effects (font (size 1 1) (thickness 0.15)) (justify mirror))
     )
-    (fp_text value Conn_02x20_Odd_Even (at -1.25 -39.25 90) (layer B.Fab)
+    (fp_text value PinSocket_2x20_P2.54mm_Vertical (at -1.25 -39.25 90) (layer B.Fab)
       (effects (font (size 1 1) (thickness 0.15)) (justify mirror))
     )
@@
       (effects (font (size 1 1) (thickness 0.15)))
     )
-    (fp_text value Screw_Terminal_01x02 (at 1.27 4.16) (layer F.Fab)
+    (fp_text value 1725656 (at 1.27 4.16) (layer F.Fab)
       (effects (font (size 1 1) (thickness 0.15)))
     )
@@
       (effects (font (size 1 1) (thickness 0.15)))
     )
-    (fp_text value Screw_Terminal_01x05 (at 6.105 0) (layer F.Fab)
+    (fp_text value 1725685 (at 6.105 0) (layer F.Fab)
       (effects (font (size 1 1) (thickness 0.15)))
     )
@@
       (effects (font (size 1 1) (thickness 0.15)))
     )
-    (fp_text value "ISP Header" (at 1.27 7.41) (layer F.Fab)
+    (fp_text value PinHeader_2x03_P2.54mm_Vertical (at 1.27 7.41) (layer F.Fab)
       (effects (font (size 1 1) (thickness 0.15)))
     )
@@
       (effects (font (size 1 1) (thickness 0.15)))
     )
-    (fp_text value FQP_27P06 (at 2.54 2.5 90) (layer F.Fab)
+    (fp_text value FQP27P06 (at 2.54 2.5 90) (layer F.Fab)
       (effects (font (size 1 1) (thickness 0.15)))
     )
@@
       (effects (font (size 1 1) (thickness 0.15)))
     )
-    (fp_text value SW_DIP_x02 (at 3.75 1.5) (layer F.Fab)
+    (fp_text value 1825057-1 (at 3.75 1.5) (layer F.Fab)
       (effects (font (size 1 1) (thickness 0.15)))
     )
@@
       (effects (font (size 1 1) (thickness 0.15)))
     )
-    (fp_text value 25LCxxx (at 0 3.68) (layer F.Fab)
+    (fp_text value 25LC1024-E/SM (at 0 3.68) (layer F.Fab)
       (effects (font (size 1 1) (thickness 0.15)))
     )
@@
       (effects (font (size 1 1) (thickness 0.15)))
     )
-    (fp_text value 8MHz (at 0 2.8) (layer F.Fab)
+    (fp_text value F90800021 (at 0 2.8) (layer F.Fab)
       (effects (font (size 1 1) (thickness 0.15)))
     )
@@
       (effects (font (size 1 1) (thickness 0.15)))
     )
-    (fp_text value 32.768kHz (at 0 1.8 90) (layer F.Fab)
-      (effects (font (size 1 1) (thickness 0.15)))
-    )
+    (fp_text value LFXTAL050789REEL (at 0 1.8 90) (layer F.Fab)
+      (effects (font (size 1 1) (thickness 0.15)))
+    )

Commit message: Add files via upload
Other:
- board text added: "12V"
- board text added: "3V3"
- board text added: "BRN"
- board text added: "GND"
- board text added: "GRN"
- board text added: "WHT"
