File: Hardware/PCB_Design/ComputationalPrototype.sch (KiCad schematic (older format))
At the start: 56 parts, among them IC1 PCF8523T_1,118, IC2 1072, J1 Conn_02x20_Odd_Even, J2 Screw_Terminal_01x02, J3 Screw_Terminal_01x05, J4 USB_B_Micro, J5 ISP Header, Q1 FQP_27P06, Q2 2N3904, SW1 SW_Push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

Commit message: Add files via upload
Parts:
- added JP?: Jumper_2_Bridged, symbol Jumper:Jumper_2_Bridged
- C4: value 1uF -> 100uF
Connections:
- wire segments 303 -> 306
Changed lines of the file:
@@
 P 3525 2575
 F 0 "C4" H 3617 2621 50  0000 L CNN
-F 1 "1uF" H 3617 2530 50  0000 L CNN
+F 1 "100uF" H 3617 2530 50  0000 L CNN
 F 2 "Capacitor_SMD:C_0805_2012Metric_Pad1.15x1.40mm_HandSolder" H 3525 2575 50  0001 C CNN
 F 3 "~" H 3525 2575 50  0001 C CNN
@@
 Wire Wire Line
 	2175 2275 2175 2425
-$Comp
-L power:+3.3V #PWR01
-U 1 1 5DD2E44B
-P 8800 1200
-F 0 "#PWR01" H 8800 1050 50  0001 C CNN
-F 1 "+3.3V" H 8815 1373 50  0000 C CNN
-F 2 "" H 8800 1200 50  0001 C CNN
-F 3 "" H 8800 1200 50  0001 C CNN
-	1    8800 1200
-	1    0    0    -1
-$EndComp
 Wire Wire Line
 	8625 6725 9275 6725
@@
 	1    0    0    -1
 $EndComp
-Wire Wire Line
-	8800 1200 8800 1225
 Connection ~ 8800 1225
 Wire Wire Line
@@
 	13175 1925 14025 1925
 Connection ~ 13175 3700
+Wire Wire Line
+	8800 810  11725 810
+Wire Wire Line
+	8800 810  8800 1225
+Wire Wire Line
+	11725 810  11725 1575
+$Comp
+L Jumper:Jumper_2_Bridged JP?
+U 1 1 60992B5E
+P 8455 810
+F 0 "JP?" H 8455 1005 50  0000 C CNN
+F 1 "Jumper_2_Bridged" H 8455 914 50  0000 C CNN
+F 2 "" H 8455 810 50  0001 C CNN
+F 3 "~" H 8455 810 50  0001 C CNN
+	1    8455 810
+	1    0    0    -1
+$EndComp
+Wire Wire Line
+	8800 810  8655 810
+Connection ~ 8800 810
 $EndSCHEMATC

Commit message: Add files via upload
Parts:
- D1, D2, D3: value LED_ALT -> 151031VS06000
- IC2: value 1072 -> Keystone 1072
- J1: value Conn_02x20_Odd_Even -> PinSocket_2x20_P2.54mm_Vertical
- J2: value Screw_Terminal_01x02 -> 1725656
- J3: value Screw_Terminal_01x05 -> 1725685
- J5: value ISP Header -> PinHeader_2x03_P2.54mm_Vertical
- JP1: renamed from JP?; value Jumper_2_Bridged -> SNT-100-YW-T; footprint (none) -> Connector_PinHeader_2.54mm:PinHeader_1x02_P2.54mm_Vertical
- Q1: value FQP_27P06 -> FQP27P06
- R12: footprint R12 -> Resistor_SMD:R_0805_2012Metric_Pad1.15x1.40mm_HandSolder
- SW1, SW2: value SW_Push -> PTS645SL432LFS
- SW3: value SW_DIP_x02 -> 1825057-1
- U1: value MCP1703A-3302_SOT23 -> MCP1703AT-3302E/CB
- U4: value 25LCxxx -> 25LC1024-E/SM
- U5: value 74125 -> SN74HC125DR
- Y1: value 8MHz -> F90800021
- Y2: value 32.768kHz -> LFXTAL050789REEL
Connections:
- wire segments 306 -> 307
Changed lines of the file:
@@
 P 8625 4875
 F 0 "SW1" V 8579 5023 50  0000 L CNN
-F 1 "SW_Push" V 8670 5023 50  0000 L CNN
+F 1 "PTS645SL432LFS" V 8670 5023 50  0000 L CNN
 F 2 "Button_Switch_THT:SW_PUSH_6mm" H 8625 5075 50  0001 C CNN
 F 3 "" H 8625 5075 50  0001 C CNN
@@
 P 6825 3775
 F 0 "Y1" V 6775 3825 50  0000 L CNN
-F 1 "8MHz" V 6975 3725 50  0000 L CNN
+F 1 "F90800021" V 6975 3725 50  0000 L CNN
 F 2 "Crystal:Crystal_SMD_Abracon_ABM3-2Pin_5.0x3.2mm" H 6825 3775 50  0001 C CNN
 F 3 "~" H 6825 3775 50  0001 C CNN
@@
 P 1625 2525
 F 0 "J2" H 1545 2200 50  0000 C CNN
-F 1 "Screw_Terminal_01x02" H 1545 2291 50  0000 C CNN
+F 1 "1725656" H 1545 2291 50  0000 C CNN
 F 2 "TerminalBlock_Phoenix:TerminalBlock_Phoenix_MPT-0,5-2-2.54_1x02_P2.54mm_Horizontal" H 1625 2525 50  0001 C CNN
 F 3 "~" H 1625 2525 50  0001 C CNN
@@
 P 2875 2425
 F 0 "U1" H 2875 2667 50  0000 C CNN
-F 1 "MCP1703A-3302_SOT23" H 2875 2576 50  0000 C CNN
+F 1 "MCP1703AT-3302E/CB" H 2875 2576 50  0000 C CNN
 F 2 "Package_TO_SOT_SMD:SOT-23_Handsoldering" H 2875 2625 50  0001 C CNN
 F 3 "http://ww1.microchip.com/downloads/en/DeviceDoc/20005122B.pdf" H 2875 2375 50  0001 C CNN
@@
 P 8025 5575
 F 0 "SW2" V 7979 5723 50  0000 L CNN
-F 1 "SW_Push" V 8070 5723 50  0000 L CNN
+F 1 "PTS645SL432LFS" V 8070 5723 50  0000 L CNN
 F 2 "Button_Switch_THT:SW_PUSH_6mm" H 8025 5775 50  0001 C CNN
 F 3 "" H 8025 5775 50  0001 C CNN
@@
 P 9175 3325
 F 0 "J3" H 9255 3367 50  0000 L CNN
-F 1 "Screw_Terminal_01x05" H 9255 3276 50  0000 L CNN
+F 1 "1725685" H 9255 3276 50  0000 L CNN
 F 2 "TerminalBlock_Phoenix:TerminalBlock_Phoenix_MPT-0,5-5-2.54_1x05_P2.54mm_Horizontal" H 9175 3325 50  0001 C CNN
 F 3 "~" H 9175 3325 50  0001 C CNN
@@
 $EndComp
 Wire Wire Line
-	8975 3425 8925 3425
-Wire Wire Line
-	8925 3425 8925 3675
-Wire Wire Line
-	8975 3525 8725 3525
-Wire Wire Line
-	8725 3525 8725 2825
-Wire Wire Line
-	8975 3325 8175 3325
-Wire Wire Line
 	8175 3325 8175 4425
 Wire Wire Line
-	8975 3225 8275 3225
-Wire Wire Line
-	8275 3225 8275 4525
-Wire Wire Line
 	8275 4525 7625 4525
 Wire Wire Line
@@
 Wire Wire Line
 	6425 5325 7825 5325
-Wire Wire Line
-	8975 3125 8375 3125
-Wire Wire Line
-	8375 3125 8375 4925
 Wire Wire Line
 	8375 4925 7725 4925
@@
 P 2325 6675
 F 0 "Y2" V 2375 6575 50  0000 R CNN
-F 1 "32.768kHz" V 2225 6675 50  0000 R CNN
+F 1 "LFXTAL050789REEL" V 2225 6675 50  0000 R CNN
 F 2 "Crystal:Crystal_SMD_2012-2Pin_2.0x1.2mm_HandSoldering" H 2325 6675 50  0001 C CNN
 F 3 "~" H 2325 6675 50  0001 C CNN
@@
 P 10650 4750
 F 0 "D1" V 10650 4650 50  0000 R CNN
-F 1 "LED_ALT" V 10597 4632 50  0001 R CNN
+F 1 "151031VS06000" V 10597 4632 50  0001 R CNN
 F 2 "LED_THT:LED_D3.0mm_Clear" H 10650 4750 50  0001 C CNN
 F 3 "~" H 10650 4750 50  0001 C CNN
@@
 P 7175 1775
 F 0 "J5" H 7225 2092 50  0000 C CNN
-F 1 "ISP Header" H 7225 2001 50  0000 C CNN
+F 1 "PinHeader_2x03_P2.54mm_Vertical" H 7225 2001 50  0000 C CNN
 F 2 "Connector_PinHeader_2.54mm:PinHeader_2x03_P2.54mm_Vertical" H 7175 1775 50  0001 C CNN
 F 3 "~" H 7175 1775 50  0001 C CNN
@@
 P 8525 9175
 F 0 "D2" V 8625 9125 50  0000 R CNN
-F 1 "LED_ALT" V 8472 9057 50  0001 R CNN
+F 1 "151031VS06000" V 8472 9057 50  0001 R CNN
 F 2 "LED_THT:LED_D3.0mm_Clear" H 8525 9175 50  0001 C CNN
 F 3 "~" H 8525 9175 50  0001 C CNN
@@
 P 8725 9175
 F 0 "D3" V 8825 9125 50  0000 R CNN
-F 1 "LED_ALT" V 8675 9075 50  0001 R CNN
+F 1 "151031VS06000" V 8675 9075 50  0001 R CNN
 F 2 "LED_THT:LED_D3.0mm_Clear" H 8725 9175 50  0001 C CNN
 F 3 "~" H 8725 9175 50  0001 C CNN
@@
 P 8525 8075
 F 0 "SW3" H 8525 8442 50  0000 C CNN
-F 1 "SW_DIP_x02" H 8525 8351 50  0000 C CNN
+F 1 "1825057-1" H 8525 8351 50  0000 C CNN
 F 2 "Button_Switch_THT:SW_DIP_SPSTx02_Slide_9.78x7.26mm_W7.62mm_P2.54mm" H 8525 8075 50  0001 C CNN
 F 3 "" H 8525 8075 50  0001 C CNN
@@
 P 8800 1600
 F 0 "U4" H 8600 1925 50  0000 C CNN
-F 1 "25LCxxx" H 8600 1850 50  0000 C CNN
+F 1 "25LC1024-E/SM" H 8600 1850 50  0000 C CNN
 F 2 "Package_SO:SOIJ-8_5.3x5.3mm_P1.27mm" H 8800 1600 50  0001 C CNN
 F 3 "http://ww1.microchip.com/downloads/en/DeviceDoc/21832H.pdf" H 8800 1600 50  0001 C CNN
@@
 P 11725 1825
 F 0 "U5" H 11725 2225 50  0000 C CNN
-F 1 "74125" H 11725 2125 50  0000 C CNN
+F 1 "SN74HC125DR" H 11725 2125 50  0000 C CNN
 F 2 "Package_SO:SOIC-14_3.9x8.7mm_P1.27mm" H 11725 1825 50  0001 C CNN
 F 3 "" H 11725 1825 50  0001 C CNN
@@
 P 11725 2600
 F 0 "U5" H 11725 3000 50  0000 C CNN
-F 1 "74125" H 11725 2900 50  0000 C CNN
+F 1 "SN74HC125DR" H 11725 2900 50  0000 C CNN
 F 2 "Package_SO:SOIC-14_3.9x8.7mm_P1.27mm" H 11725 2600 50  0001 C CNN
 F 3 "" H 11725 2600 50  0001 C CNN
@@
 P 11725 3375
 F 0 "U5" H 11725 3775 50  0000 C CNN
-F 1 "74125" H 11725 3675 50  0000 C CNN
+F 1 "SN74HC125DR" H 11725 3675 50  0000 C CNN
 F 2 "Package_SO:SOIC-14_3.9x8.7mm_P1.27mm" H 11725 3375 50  0001 C CNN
 F 3 "" H 11725 3375 50  0001 C CNN
@@
 P 11725 4150
 F 0 "U5" H 11725 4550 50  0000 C CNN
-F 1 "74125" H 11725 4450 50  0000 C CNN
+F 1 "SN74HC125DR" H 11725 4450 50  0000 C CNN
 F 2 "Package_SO:SOIC-14_3.9x8.7mm_P1.27mm" H 11725 4150 50  0001 C CNN
 F 3 "" H 11725 4150 50  0001 C CNN
@@
 P 12325 5425
 F 0 "Q1" H 12530 5379 50  0000 L CNN
-F 1 "FQP_27P06" H 12530 5470 50  0000 L CNN
+F 1 "FQP27P06" H 12530 5470 50  0000 L CNN
 F 2 "Package_TO_SOT_THT:TO-220-3_Vertical" H 12525 5525 50  0001 C CNN
 F 3 "~" H 12325 5425 50  0001 C CNN
@@
 P 2400 7200
 F 0 "IC2" V 2754 7841 50  0000 L CNN
-F 1 "1072" V 2845 7841 50  0000 L CNN
+F 1 "Keystone 1072" V 2845 7841 50  0000 L CNN
 F 2 "1072" H 3050 7600 50  0001 L CNN
 F 3 "http://www.keystoneelectronics.net/ENG._DEPT/WEB_ORACLE/PDF/PDF%20CAT%20NO%20DRAWINGS/1000-1999/1072.PDF" H 3050 7500 50  0001 L CNN
@@
 F 0 "R12" V 12795 5125 50  0000 C CNN
 F 1 "2k" V 12886 5125 50  0000 C CNN
-F 2 "R12" H 13000 5125 50  0000 C CNN
+F 2 "Resistor_SMD:R_0805_2012Metric_Pad1.15x1.40mm_HandSolder" H 13085 5220 50  0001 C CNN
 F 3 "~" H 13000 5125 50  0001 C CNN
 	1    13000 5125
@@
 P 14225 2825
 F 0 "J1" H 14275 3942 50  0000 C CNN
-F 1 "Conn_02x20_Odd_Even" H 14275 3851 50  0000 C CNN
+F 1 "PinSocket_2x20_P2.54mm_Vertical" H 14275 3851 50  0000 C CNN
 F 2 "Connector_PinSocket_2.54mm:PinSocket_2x20_P2.54mm_Vertical" H 14225 2825 50  0001 C CNN
 F 3 "~" H 14225 2825 50  0001 C CNN
@@
 	11725 810  11725 1575
 $Comp
-L Jumper:Jumper_2_Bridged JP?
+L Jumper:Jumper_2_Bridged JP1
 U 1 1 60992B5E
 P 8455 810
-F 0 "JP?" H 8455 1005 50  0000 C CNN
-F 1 "Jumper_2_Bridged" H 8455 914 50  0000 C CNN
-F 2 "" H 8455 810 50  0001 C CNN
+F 0 "JP1" H 8455 1005 50  0000 C CNN
+F 1 "SNT-100-YW-T" H 8455 914 50  0000 C CNN
+F 2 "Connector_PinHeader_2.54mm:PinHeader_1x02_P2.54mm_Vertical" H 8455 810 50  0001 C CNN
 F 3 "~" H 8455 810 50  0001 C CNN
 	1    8455 810
@@
 	8800 810  8655 810
 Connection ~ 8800 810
+Wire Wire Line
+	8975 3125 8725 3125
+Wire Wire Line
+	8725 3125 8725 2825
+Wire Wire Line
+	8925 3225 8975 3225
+Wire Wire Line
+	8925 3225 8925 3675
+Wire Wire Line
+	8375 3525 8375 4925
+Wire Wire Line
+	8975 3425 8275 3425
+Wire Wire Line
+	8275 3425 8275 4525
+Wire Wire Line
+	8175 3325 8975 3325
+Wire Wire Line
+	8375 3525 8975 3525
+Wire Wire Line
+	8255 810  8020 810
+$Comp
+L power:+3.3V #PWR0108
+U 1 1 609F3650
+P 8020 810
+F 0 "#PWR0108" H 8020 660 50  0001 C CNN
+F 1 "+3.3V" H 8035 983 50  0000 C CNN
+F 2 "" H 8020 810 50  0001 C CNN
+F 3 "" H 8020 810 50  0001 C CNN
+	1    8020 810
+	1    0    0    -1
+$EndComp
 $EndSCHEMATC
